File: unix69/kicad/keybird.kicad_sch (KiCad schematic)
At the start: 139 parts, among them SW00 ESC, SW01 2, SW02 4, SW03 6, SW04 8, SW05 0, SW06 EQUAL, SW07 GRAVE, SW10 1, SW11 3, SW12 5, SW13 7, SW14 9, SW15 MINUS, SW16 BSLS, SW17 F16, SW20 TAB, SW21 W, SW22 R, SW23 Y, SW24 I, SW25 P, SW26 RBRC, SW27 F17, SW30 Q, SW31 E, SW32 T, SW33 U, SW34 O, SW35 LBRC, SW36 BSPC, SW40 A, SW41 D, SW42 G, SW43 J, SW44 L, SW45 QUOTE, SW47 F18, SW50 LCTL, SW51 S, SW52 F, SW53 H, SW54 K, SW55 SCLN, SW56 ENTER, SW57 F19, SW60 LSFT, SW61 X, SW62 V, SW63 N, SW64 COMMA, SW65 SLASH, SW66 RSFT, SW67 UP, SW70 LFN, SW71 Z, SW72 C, SW73 B, SW74 M, SW75 DOT, SW76 LEFT, SW77 RIGHT, SW80 LALT, SW81 LGUI, SW83 SPACE, SW84 RGUI, SW85 RCTL, SW86 RFN, SW87 DOWN, U2040 RP2040-Tiny

Commit message: major revision
Parts:
- removed D75: DIODE, Diode_SMD:D_SOD-123, symbol pspice:DIODE
- removed SW75: DOT, Switch_Keyboard_Hotswap_Kailh:SW_Hotswap_Kailh_MX_1.00u, symbol Switch:SW_Push
- added D82: DIODE, Diode_SMD:D_SOD-123, symbol pspice:DIODE
- added SW82: LMETA, Switch_Keyboard_Hotswap_Kailh:SW_Hotswap_Kailh_MX_1.25u, symbol Switch:SW_Push
- SW07: value GRAVE -> BQUOT
- SW16: value BSLS -> BSLSH
- SW17: value F16 -> F13
- SW26: value RBRC -> RBRAC
- SW27: value F17 -> F14
- SW35: value LBRC -> LBRAC
- SW36: value BSPC -> DEL
- SW47: value F18 -> F15
- SW50: value LCTL -> LCTRL
- SW55: value SCLN -> COLON
- SW56: value ENTER -> RET
- SW57: value F19 -> F16
- SW60: value LSFT -> LSHFT
- SW66: value RSFT -> RSHFT
- SW70: value LFN -> Z; footprint Switch_Keyboard_Hotswap_Kailh:SW_Hotswap_Kailh_MX_1.25u -> Switch_Keyboard_Hotswap_Kailh:SW_Hotswap_Kailh_MX_1.00u
- SW71: value Z -> C
- SW72: value C -> B
- SW73: value B -> M
- SW74: value M -> DOT
- SW80: value LALT -> LFUN
- SW81: value LGUI -> LALT
- SW84: value RGUI -> RMETA
- SW85: value RCTL -> RCTRL
- SW86: value RFN -> RFUN
- renumbered U2040 to U1
Connections:
- net COL0: now also SW00.2, SW10.2, SW20.2, SW30.2, SW40.2, SW50.2, SW60.2, SW70.2, SW80.2, U1.0 (GP0); no longer SW00.1, SW10.1, SW20.1, SW30.1, SW40.1, SW50.1, SW60.1, SW70.1, SW80.1, U1.14 (GP14)
- net COL1: now also SW01.2, SW11.2, SW21.2, SW31.2, SW41.2, SW51.2, SW61.2, SW71.2, SW81.2, U1.1 (GP1); no longer SW01.1, SW11.1, SW21.1, SW31.1, SW41.1, SW51.1, SW61.1, SW71.1, SW81.1, U1.15 (GP15)
- net COL2: now also SW02.2, SW12.2, SW22.2, SW32.2, SW42.2, SW52.2, SW62.2, SW72.2, U1.2 (GP2), SW82.2; no longer SW02.1, SW12.1, SW22.1, SW32.1, SW42.1, SW52.1, SW62.1, SW72.1, U1.16 (GP26)
- net COL3: now also SW03.2, SW13.2, SW23.2, SW33.2, SW43.2, SW53.2, SW63.2, SW73.2, SW83.2, U1.3 (GP3); no longer SW03.1, SW13.1, SW23.1, SW33.1, SW43.1, SW53.1, SW63.1, SW73.1, SW83.1, U1.13 (GP13)
- net COL4: now also SW04.2, SW14.2, SW24.2, SW34.2, SW44.2, SW54.2, SW64.2, SW74.2, SW84.2, U1.7 (GP7); no longer SW04.1, SW14.1, SW24.1, SW34.1, SW44.1, SW54.1, SW64.1, SW74.1, SW84.1, U1.12 (GP12)
- net COL5: now also SW05.2, SW15.2, SW25.2, SW35.2, SW45.2, SW55.2, SW65.2, SW85.2, U1.6 (GP6); no longer SW05.1, SW15.1, SW25.1, SW35.1, SW45.1, SW55.1, SW65.1, SW85.1, U1.11 (GP11)
- net COL6: now also SW06.2, SW16.2, SW26.2, SW36.2, SW56.2, SW66.2, SW76.2, SW86.2, U1.5 (GP5); no longer SW06.1, SW16.1, SW26.1, SW36.1, SW56.1, SW66.1, SW76.1, SW86.1, U1.10 (GP10)
- net COL7: now also SW07.2, SW17.2, SW27.2, SW47.2, SW57.2, SW67.2, SW77.2, SW87.2, U1.4 (GP4); no longer SW07.1, SW17.1, SW27.1, SW47.1, SW57.1, SW67.1, SW77.1, SW87.1, U1.9 (GP9)
- net ROW0: now also U1.9 (GP9); no longer U1.0 (GP0)
- net ROW1: now also U1.10 (GP10); no longer U1.1 (GP1)
- net ROW2: now also U1.11 (GP11); no longer U1.2 (GP2)
- net ROW3: now also U1.12 (GP12); no longer U1.3 (GP3)
- net ROW4: now also U1.13 (GP13); no longer U1.4 (GP4)
- net ROW5: now also U1.14 (GP14); no longer U1.5 (GP5)
- net ROW6: now also U1.15 (GP15); no longer U1.6 (GP6)
- net ROW7: now also U1.16 (GP26); no longer U1.7 (GP7)
- net ROW8: now also D82.2 (A)
- net at D81.1 (K): now also SW81.1; no longer SW81.2
- net at D41.1 (K): now also SW41.1; no longer SW41.2
- net at D04.1 (K): now also SW04.1; no longer SW04.2
- net at D52.1 (K): now also SW52.1; no longer SW52.2
- net at D64.1 (K): now also SW64.1; no longer SW64.2
- net at D84.1 (K): now also SW84.1; no longer SW84.2
- net at D06.1 (K): now also SW06.1; no longer SW06.2
- net at D53.1 (K): now also SW53.1; no longer SW53.2
- net at D56.1 (K): now also SW56.1; no longer SW56.2
- net at D44.1 (K): now also SW44.1; no longer SW44.2
- net at D30.1 (K): now also SW30.1; no longer SW30.2
- net at D62.1 (K): now also SW62.1; no longer SW62.2
- net at D67.1 (K): now also SW67.1; no longer SW67.2
- net at D33.1 (K): now also SW33.1; no longer SW33.2
- net at D72.1 (K): now also SW72.1; no longer SW72.2
- net at D22.1 (K): now also SW22.1; no longer SW22.2
- net at D25.1 (K): now also SW25.1; no longer SW25.2
- net at D35.1 (K): now also SW35.1; no longer SW35.2
- net at D66.1 (K): now also SW66.1; no longer SW66.2
- net at D12.1 (K): now also SW12.1; no longer SW12.2
- net at D20.1 (K): now also SW20.1; no longer SW20.2
- net at D00.1 (K): now also SW00.1; no longer SW00.2
- net at D03.1 (K): now also SW03.1; no longer SW03.2
- net at D10.1 (K): now also SW10.1; no longer SW10.2
- net at D63.1 (K): now also SW63.1; no longer SW63.2
- net at D26.1 (K): now also SW26.1; no longer SW26.2
- net at D87.1 (K): now also SW87.1; no longer SW87.2
- net at D54.1 (K): now also SW54.1; no longer SW54.2
- net at D73.1 (K): now also SW73.1; no longer SW73.2
- net at D01.1 (K): now also SW01.1; no longer SW01.2
- net at D71.1 (K): now also SW71.1; no longer SW71.2
- net at D13.1 (K): now also SW13.1; no longer SW13.2
- net at D60.1 (K): now also SW60.1; no longer SW60.2
- net at D42.1 (K): now also SW42.1; no longer SW42.2
- net at D34.1 (K): now also SW34.1; no longer SW34.2
- net at D70.1 (K): now also SW70.1; no longer SW70.2
- net at D83.1 (K): now also SW83.1; no longer SW83.2
- net at D55.1 (K): now also SW55.1; no longer SW55.2
- net at D45.1 (K): now also SW45.1; no longer SW45.2
- net at D14.1 (K): now also SW14.1; no longer SW14.2
- net at D61.1 (K): now also SW61.1; no longer SW61.2
- net at D36.1 (K): now also SW36.1; no longer SW36.2
- net at D77.1 (K): now also SW77.1; no longer SW77.2
- net at D85.1 (K): now also SW85.1; no longer SW85.2
- net at D40.1 (K): now also SW40.1; no longer SW40.2
- net at D24.1 (K): now also SW24.1; no longer SW24.2
- net at D57.1 (K): now also SW57.1; no longer SW57.2
- net at D47.1 (K): now also SW47.1; no longer SW47.2
- net at D07.1 (K): now also SW07.1; no longer SW07.2
- net at D05.1 (K): now also SW05.1; no longer SW05.2
- net at D15.1 (K): now also SW15.1; no longer SW15.2
- net at D23.1 (K): now also SW23.1; no longer SW23.2
- net at D51.1 (K): now also SW51.1; no longer SW51.2
- net at D65.1 (K): now also SW65.1; no longer SW65.2
- net at D17.1 (K): now also SW17.1; no longer SW17.2
- net at D02.1 (K): now also SW02.1; no longer SW02.2
- net at D86.1 (K): now also SW86.1; no longer SW86.2
- net at D76.1 (K): now also SW76.1; no longer SW76.2
- net at D27.1 (K): now also SW27.1; no longer SW27.2
- net at D16.1 (K): now also SW16.1; no longer SW16.2
- net at D21.1 (K): now also SW21.1; no longer SW21.2
- net at D50.1 (K): now also SW50.1; no longer SW50.2
- net at D80.1 (K): now also SW80.1; no longer SW80.2
- net at D32.1 (K): now also SW32.1; no longer SW32.2
- net at D11.1 (K): now also SW11.1; no longer SW11.2
- net at D74.1 (K): now also SW74.1; no longer SW74.2
- net at D31.1 (K): now also SW31.1; no longer SW31.2
- net at D43.1 (K): now also SW43.1; no longer SW43.2
- new net: D82.1 (K), SW82.1
- no-connect marks 79 -> 77
