File: unix69/kicad/keybird.kicad_sch (KiCad schematic)
At the start: 139 parts, among them SW00 ESC, SW01 2, SW02 4, SW03 6, SW04 8, SW05 0, SW06 EQUAL, SW07 BQUOT, SW10 1, SW11 3, SW12 5, SW13 7, SW14 9, SW15 MINUS, SW16 BSLSH, SW17 F13, SW20 TAB, SW21 W, SW22 R, SW23 Y, SW24 I, SW25 P, SW26 RBRAC, SW27 F14, SW30 Q, SW31 E, SW32 T, SW33 U, SW34 O, SW35 LBRAC, SW36 DEL, SW40 A, SW41 D, SW42 G, SW43 J, SW44 L, SW45 QUOTE, SW47 F15, SW50 LCTRL, SW51 S, SW52 F, SW53 H, SW54 K, SW55 COLON, SW56 RET, SW57 F16, SW60 LSHFT, SW61 X, SW62 V, SW63 N, SW64 COMMA, SW65 SLASH, SW66 RSHFT, SW67 UP, SW70 Z, SW71 C, SW72 B, SW73 M, SW74 DOT, SW76 LEFT, SW77 RIGHT, SW80 LFUN, SW81 LALT, SW82 LMETA, SW83 SPACE, SW84 RMETA, SW85 RCTRL, SW86 RFUN, SW87 DOWN, U1 RP2040-Tiny

Commit message: very nice, i think
Changed lines of the file:
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@@
   (no_connect (at 165.1 139.7))
   (no_connect (at 63.5 88.9))
-  (no_connect (at 66.04 153.67))
+  (no_connect (at 71.12 152.4))
   (no_connect (at 114.3 101.6))
   (no_connect (at 190.5 63.5))
@@
   (no_connect (at 190.5 88.9))
   (no_connect (at 165.1 114.3))
-  (no_connect (at 73.66 153.67))
+  (no_connect (at 78.74 152.4))
   (no_connect (at 38.1 63.5))
   (no_connect (at 165.1 101.6))
@@
   (no_connect (at 215.9 101.6))
   (no_connect (at 190.5 139.7))
-  (no_connect (at 58.42 153.67))
+  (no_connect (at 63.5 152.4))
   (no_connect (at 88.9 127))
-  (no_connect (at 62.23 153.67))
-  (no_connect (at 54.61 153.67))
+  (no_connect (at 67.31 152.4))
+  (no_connect (at 59.69 152.4))
   (no_connect (at 190.5 76.2))
   (no_connect (at 114.3 76.2))
@@
     (stroke (width 0) (type default) (color 0 0 0 0))
   )
-  (wire (pts (xy 31.75 167.64) (xy 38.1 167.64))
+  (wire (pts (xy 31.75 161.29) (xy 38.1 161.29))
     (stroke (width 0) (type default) (color 0 0 0 0))
   )
@@
     (stroke (width 0) (type default) (color 0 0 0 0))
   )
-  (wire (pts (xy 54.61 189.23) (xy 54.61 195.58))
+  (wire (pts (xy 59.69 177.8) (xy 59.69 184.15))
     (stroke (width 0) (type default) (color 0 0 0 0))
   )
@@
     (stroke (width 0) (type default) (color 0 0 0 0))
   )
-  (wire (pts (xy 31.75 179.07) (xy 38.1 179.07))
+  (wire (pts (xy 31.75 172.72) (xy 38.1 172.72))
     (stroke (width 0) (type default) (color 0 0 0 0))
   )
@@
     (stroke (width 0) (type default) (color 0 0 0 0))
   )
-  (wire (pts (xy 58.42 189.23) (xy 58.42 195.58))
+  (wire (pts (xy 63.5 177.8) (xy 63.5 184.15))
     (stroke (width 0) (type default) (color 0 0 0 0))
   )
@@
     (stroke (width 0) (type default) (color 0 0 0 0))
   )
-  (wire (pts (xy 69.85 195.58) (xy 69.85 189.23))
+  (wire (pts (xy 74.93 184.15) (xy 74.93 177.8))
     (stroke (width 0) (type default) (color 0 0 0 0))
   )
@@
     (stroke (width 0) (type default) (color 0 0 0 0))
   )
-  (wire (pts (xy 31.75 163.83) (xy 38.1 163.83))
+  (wire (pts (xy 31.75 157.48) (xy 38.1 157.48))
     (stroke (width 0) (type default) (color 0 0 0 0))
   )
@@
     (stroke (width 0) (type default) (color 0 0 0 0))
   )
-  (wire (pts (xy 31.75 171.45) (xy 38.1 171.45))
+  (wire (pts (xy 31.75 165.1) (xy 38.1 165.1))
     (stroke (width 0) (type default) (color 0 0 0 0))
   )
@@
     (stroke (width 0) (type default) (color 0 0 0 0))
   )
-  (wire (pts (xy 31.75 175.26) (xy 38.1 175.26))
+  (wire (pts (xy 31.75 168.91) (xy 38.1 168.91))
     (stroke (width 0) (type default) (color 0 0 0 0))
   )
@@
     (stroke (width 0) (type default) (color 0 0 0 0))
   )
-  (wire (pts (xy 46.99 189.23) (xy 46.99 195.58))
+  (wire (pts (xy 52.07 177.8) (xy 52.07 184.15))
     (stroke (width 0) (type default) (color 0 0 0 0))
   )
@@
     (stroke (width 0) (type default) (color 0 0 0 0))
   )
-  (wire (pts (xy 50.8 189.23) (xy 50.8 195.58))
+  (wire (pts (xy 55.88 177.8) (xy 55.88 184.15))
     (stroke (width 0) (type default) (color 0 0 0 0))
   )
@@
     (stroke (width 0) (type default) (color 0 0 0 0))
   )
-  (wire (pts (xy 73.66 195.58) (xy 73.66 189.23))
+  (wire (pts (xy 78.74 184.15) (xy 78.74 177.8))
     (stroke (width 0) (type default) (color 0 0 0 0))
   )
@@
     (stroke (width 0) (type default) (color 0 0 0 0))
   )
-  (wire (pts (xy 46.99 147.32) (xy 46.99 153.67))
+  (wire (pts (xy 52.07 146.05) (xy 52.07 152.4))
     (stroke (width 0) (type default) (color 0 0 0 0))
   )
@@
     (stroke (width 0) (type default) (color 0 0 0 0))
   )
-  (wire (pts (xy 43.18 195.58) (xy 43.18 189.23))
+  (wire (pts (xy 48.26 184.15) (xy 48.26 177.8))
     (stroke (width 0) (type default) (color 0 0 0 0))
   )
@@
     (stroke (width 0) (type default) (color 0 0 0 0))
   )
-  (wire (pts (xy 66.04 195.58) (xy 66.04 189.23))
+  (wire (pts (xy 71.12 184.15) (xy 71.12 177.8))
     (stroke (width 0) (type default) (color 0 0 0 0))
   )
@@
     (stroke (width 0) (type default) (color 0 0 0 0))
   )
-  (wire (pts (xy 43.18 147.32) (xy 43.18 153.67))
+  (wire (pts (xy 48.26 146.05) (xy 48.26 152.4))
     (stroke (width 0) (type default) (color 0 0 0 0))
   )
@@
     (stroke (width 0) (type default) (color 0 0 0 0))
   )
-  (wire (pts (xy 50.8 147.32) (xy 50.8 153.67))
+  (wire (pts (xy 55.88 146.05) (xy 55.88 152.4))
     (stroke (width 0) (type default) (color 0 0 0 0))
   )
@@
     (stroke (width 0) (type default) (color 0 0 0 0))
   )
-  (wire (pts (xy 62.23 189.23) (xy 62.23 195.58))
+  (wire (pts (xy 67.31 177.8) (xy 67.31 184.15))
     (stroke (width 0) (type default) (color 0 0 0 0))
   )
@@
     (effects (font (size 1.27 1.27)) (justify left bottom))
   )
-  (label "ROW5" (at 43.18 147.32 270)
+  (label "ROW5" (at 48.26 146.05 270)
     (effects (font (size 1.27 1.27)) (justify right bottom))
   )
-  (label "ROW7" (at 50.8 147.32 270)
+  (label "ROW7" (at 55.88 146.05 270)
     (effects (font (size 1.27 1.27)) (justify right bottom))
   )
-  (label "COL5" (at 50.8 195.58 90)
+  (label "COL5" (at 55.88 184.15 90)
     (effects (font (size 1.27 1.27)) (justify left bottom))
   )
@@
     (effects (font (size 1.27 1.27)) (justify left bottom))
   )
-  (label "COL4" (at 46.99 195.58 90)
-    (effects (font (size 1.27 1.27)) (justify left bottom))
-  )
-  (label "ROW2" (at 31.75 171.45 0)
-    (effects (font (size 1.27 1.27)) (justify left bottom))
-  )
-  (label "ROW4" (at 31.75 163.83 0)
+  (label "COL4" (at 52.07 184.15 90)
+    (effects (font (size 1.27 1.27)) (justify left bottom))
+  )
+  (label "ROW2" (at 31.75 165.1 0)
+    (effects (font (size 1.27 1.27)) (justify left bottom))
+  )
+  (label "ROW4" (at 31.75 157.48 0)
     (effects (font (size 1.27 1.27)) (justify left bottom))
   )
@@
     (effects (font (size 1.27 1.27)) (justify left bottom))
   )
-  (label "ROW1" (at 31.75 175.26 0)
+  (label "ROW1" (at 31.75 168.91 0)
     (effects (font (size 1.27 1.27)) (justify left bottom))
   )
@@
     (effects (font (size 1.27 1.27)) (justify left bottom))
   )
-  (label "COL1" (at 69.85 195.58 90)
-    (effects (font (size 1.27 1.27)) (justify left bottom))
-  )
-  (label "ROW6" (at 46.99 147.32 270)
+  (label "COL1" (at 74.93 184.15 90)
+    (effects (font (size 1.27 1.27)) (justify left bottom))
+  )
+  (label "ROW6" (at 52.07 146.05 270)
     (effects (font (size 1.27 1.27)) (justify right bottom))
   )
-  (label "ROW8" (at 43.18 195.58 90)
-    (effects (font (size 1.27 1.27)) (justify left bottom))
-  )
-  (label "COL7" (at 58.42 195.58 90)
+  (label "ROW8" (at 48.26 184.15 90)
+    (effects (font (size 1.27 1.27)) (justify left bottom))
+  )
+  (label "COL7" (at 63.5 184.15 90)
     (effects (font (size 1.27 1.27)) (justify left bottom))
   )
@@
     (effects (font (size 1.27 1.27)) (justify left bottom))
   )
-  (label "ROW3" (at 31.75 167.64 0)
-    (effects (font (size 1.27 1.27)) (justify left bottom))
-  )
-  (label "COL3" (at 62.23 195.58 90)
+  (label "ROW3" (at 31.75 161.29 0)
+    (effects (font (size 1.27 1.27)) (justify left bottom))
+  )
+  (label "COL3" (at 67.31 184.15 90)
     (effects (font (size 1.27 1.27)) (justify left bottom))
   )
@@
     (effects (font (size 1.27 1.27)) (justify left bottom))
   )
-  (label "COL6" (at 54.61 195.58 90)
-    (effects (font (size 1.27 1.27)) (justify left bottom))
-  )
-  (label "COL2" (at 66.04 195.58 90)
+  (label "COL6" (at 59.69 184.15 90)
+    (effects (font (size 1.27 1.27)) (justify left bottom))
+  )
+  (label "COL2" (at 71.12 184.15 90)
     (effects (font (size 1.27 1.27)) (justify left bottom))
   )
@@
     (effects (font (size 1.27 1.27)) (justify left bottom))
   )
-  (label "ROW0" (at 31.75 179.07 0)
-    (effects (font (size 1.27 1.27)) (justify left bottom))
-  )
-  (label "COL0" (at 73.66 195.58 90)
+  (label "ROW0" (at 31.75 172.72 0)
+    (effects (font (size 1.27 1.27)) (justify left bottom))
+  )
+  (label "COL0" (at 78.74 184.15 90)
     (effects (font (size 1.27 1.27)) (justify left bottom))
   )
@@
     (pin "2")
   )
-  (symbol (lib_id "MCU_Module:RP2040-Tiny") (at 57.15 171.45 180) (unit 1)
+  (symbol (lib_id "MCU_Module:RP2040-Tiny") (at 62.23 165.1 180) (unit 1)
     (in_bom yes) (on_board yes)
-    (property "Reference" "U1" (id 0) (at 57.15 172.72 0))
-    (property "Value" "RP2040-Tiny" (id 1) (at 63.5 170.18 0)
+    (property "Reference" "U1" (id 0) (at 62.23 166.37 0))
+    (property "Value" "RP2040-Tiny" (id 1) (at 68.58 163.83 0)
       (effects (font (size 1.27 1.27)) (justify left))
     )
-    (property "Footprint" "Module:RP2040-Tiny" (id 2) (at 57.15 168.91 0)
-      (effects (font (size 1.27 1.27)) hide)
-    )
-    (property "Datasheet" "" (id 3) (at 57.15 171.45 0)
+    (property "Footprint" "Module:RP2040-Tiny" (id 2) (at 62.23 162.56 0)
+      (effects (font (size 1.27 1.27)) hide)
+    )
+    (property "Datasheet" "" (id 3) (at 62.23 165.1 0)
       (effects (font (size 1.27 1.27)) hide)
     )
@@
     (pin "2")
   )
-  (symbol (lib_id "power:GND") (at 69.85 153.67 180) (unit 1)
-    (in_bom yes) (on_board yes) (fields_autoplaced)
-    (property "Reference" "#PWR0101" (id 0) (at 69.85 147.32 0)
-      (effects (font (size 1.27 1.27)) hide)
-    )
-    (property "Value" "GND" (id 1) (at 69.85 148.59 0))
-    (property "Footprint" "" (id 2) (at 69.85 153.67 0)
-      (effects (font (size 1.27 1.27)) hide)
-    )
-    (property "Datasheet" "" (id 3) (at 69.85 153.67 0)
-      (effects (font (size 1.27 1.27)) hide)
-    )
+  (symbol (lib_id "power:GND") (at 74.93 152.4 180) (unit 1)
+    (in_bom yes) (on_board yes) (fields_autoplaced)
+    (property "Reference" "#PWR0101" (id 0) (at 74.93 146.05 0)
+      (effects (font (size 1.27 1.27)) hide)
+    )
+    (property "Value" "GND" (id 1) (at 74.93 147.32 0))
+    (property "Footprint" "" (id 2) (at 74.93 152.4 0)
+      (effects (font (size 1.27 1.27)) hide)
+    )
+    (property "Datasheet" "" (id 3) (at 74.93 152.4 0)
+      (effects (font (size 1.27 1.27)) hide)
+    )

Commit message: update
Parts:
- SW56: value RET -> RETURN
Changed lines of the file:
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@@
+    (pin "2")
+  )
+  (symbol (lib_id "pspice:DIODE") (at 154.94 96.52 0) (unit 1)
+    (in_bom yes) (on_board yes) (fields_autoplaced)
+    (property "Reference" "D54" (id 0) (at 154.94 91.44 0))
+    (property "Value" "DIODE" (id 1) (at 154.94 100.965 0)
+      (effects (font (size 1.27 1.27)) hide)
+    )
+    (property "Footprint" "Diode_SMD:D_SOD-123" (id 2) (at 154.94 96.52 0)
+      (effects (font (size 1.27 1.27)) hide)
+    )
+    (property "Datasheet" "~" (id 3) (at 154.94 96.52 0)
+      (effects (font (size 1.27 1.27)) hide)
+    )
+    (pin "1")
     (pin "2")
   )
@@
     (in_bom yes) (on_board yes) (fields_autoplaced)
     (property "Reference" "SW56" (id 0) (at 195.58 91.44 0))
-    (property "Value" "RET" (id 1) (at 195.58 98.044 0))
+    (property "Value" "RETURN" (id 1) (at 195.58 98.044 0))
     (property "Footprint" "Switch_Keyboard_Hotswap_Kailh:SW_Hotswap_Kailh_MX_2.25u" (id 2) (at 195.58 91.44 0)
       (effects (font (size 1.27 1.27)) hide)
@@
     )
     (property "Datasheet" "~" (id 3) (at 231.14 134.62 0)
-      (effects (font (size 1.27 1.27)) hide)
-    )
-    (pin "1")
-    (pin "2")
-  )
-  (symbol (lib_name "DIODE_1") (lib_id "pspice:DIODE") (at 154.94 96.52 0) (unit 1)
-    (in_bom yes) (on_board yes) (fields_autoplaced)
-    (property "Reference" "D54" (id 0) (at 154.94 91.44 0))
-    (property "Value" "DIODE" (id 1) (at 154.94 100.965 0)
-      (effects (font (size 1.27 1.27)) hide)
-    )
-    (property "Footprint" "Diode_SMD:D_SOD-123" (id 2) (at 154.94 96.52 0)
-      (effects (font (size 1.27 1.27)) hide)
-    )
-    (property "Datasheet" "~" (id 3) (at 154.94 96.52 0)
       (effects (font (size 1.27 1.27)) hide)
     )
@@
       (reference "D53") (unit 1) (value "DIODE") (footprint "Diode_SMD:D_SOD-123")
     )
-    (path "/2f7398cb-95ae-49e6-9237-a3d045dca7a5"
+    (path "/0cf4c8e4-24f5-43c2-a806-52aadffe961d"
       (reference "D54") (unit 1) (value "DIODE") (footprint "Diode_SMD:D_SOD-123")
     )
@@
     )
     (path "/11aa4558-7006-4da7-9142-6a23f41bab44"
-      (reference "SW56") (unit 1) (value "RET") (footprint "Switch_Keyboard_Hotswap_Kailh:SW_Hotswap_Kailh_MX_2.25u")
+      (reference "SW56") (unit 1) (value "RETURN") (footprint "Switch_Keyboard_Hotswap_Kailh:SW_Hotswap_Kailh_MX_2.25u")
     )
     (path "/6cb32a04-e4e5-4471-bd17-7b5f8deb63bb"

Commit message: move edited library footprints into the project
Parts:
- SW00, SW01, SW02, SW03, SW04, SW05, SW06, SW07, SW10, SW11, SW12, SW13, SW14, SW15, SW16, SW17, SW21, SW22, SW23, SW24, SW25, SW26, SW27, SW30, SW31, SW32, SW33, SW34, SW35, SW40, SW41, SW42, SW43, SW44, SW45, SW47, SW51, SW52, SW53, SW54, SW55, SW57, SW61, SW62, SW63, SW64, SW65, SW67, SW70, SW71, SW72, SW73, SW74, SW76, SW77, SW84, SW85, SW86, SW87: footprint Switch_Keyboard_Hotswap_Kailh:SW_Hotswap_Kailh_MX_1.00u -> Keybird:SW_Hotswap_Kailh_MX_1.00u
- SW20, SW36: footprint Switch_Keyboard_Hotswap_Kailh:SW_Hotswap_Kailh_MX_1.50u -> Keybird:SW_Hotswap_Kailh_MX_1.50u
- SW50, SW66: footprint Switch_Keyboard_Hotswap_Kailh:SW_Hotswap_Kailh_MX_1.75u -> Keybird:SW_Hotswap_Kailh_MX_1.75u
- SW56, SW60: footprint Switch_Keyboard_Hotswap_Kailh:SW_Hotswap_Kailh_MX_2.25u -> Keybird:SW_Hotswap_Kailh_MX_2.25u
- SW83: footprint Switch_Keyboard_Hotswap_Kailh:SW_Hotswap_Kailh_MX_6.25u -> Keybird:SW_Hotswap_Kailh_MX_6.25u
