File: unix69/kicad/keybird.kicad_pcb (KiCad board)
At the start: 2 copper layers, 304.8 x 95.2 mm, 142 parts, among them SW00 ESC, SW01 2, SW02 4, SW03 6, SW04 8, SW05 0, SW06 EQUAL, SW07 BQUOT, SW10 1, SW11 3, SW12 5, SW13 7, SW14 9, SW15 MINUS, SW16 BSLSH, SW17 F13, SW20 TAB, SW21 W, SW22 R, SW23 Y, SW24 I, SW25 P, SW26 RBRAC, SW27 F14, SW30 Q, SW31 E, SW32 T, SW33 U, SW34 O, SW35 LBRAC, SW36 DEL, SW40 A, SW41 D, SW42 G, SW43 J, SW44 L, SW45 QUOTE, SW47 F15, SW50 LCTRL, SW51 S, SW52 F, SW53 H, SW54 K, SW55 COLON, SW56 RET, SW57 F16, SW60 LSHFT, SW61 X, SW62 V, SW63 N, SW64 COMMA, SW65 SLASH, SW66 RSHFT, SW67 UP, SW70 Z, SW71 C, SW72 B, SW73 M, SW74 DOT, SW76 LEFT, SW77 RIGHT, SW80 LFUN, SW81 LALT, SW82 LMETA, SW83 SPACE, SW84 RMETA, SW85 RCTRL, SW86 RFUN, SW87 DOWN, U1 RP2040-Tiny

Commit message: add ground planes
with stripes!
Routing:
- net GND: vias 0 -> 8
- added copper zone on B.Cu, net GND
- added copper zone on F.Cu, net GND

Commit message: update
Parts:
- SW56: value RET -> RETURN
Routing:
- net /COL4: track 307.2 -> 304.4 mm
- net /COL3: track 223.5 -> 220.7 mm
Other:
- board text added: "0.2"
- board text removed: "rev 0.2"

Commit message: remove usb cutout from pcb
i lack the effort for a bigger revision
Parts:
- moved D13 15.7 mm to (150.0, 26.1)
- moved D04 15.7 mm to (169.1, 26.3)
- moved D00 4.67 mm to (16.7, 26.2)
- moved D06 4.67 mm to (245.3, 26.2)
- moved D10 4.67 mm to (35.7, 26.2)
- moved D16 4.67 mm to (264.3, 26.1)
- moved D01 4.67 mm to (54.8, 26.2)
- moved D02 4.67 mm to (92.9, 26.2)
- moved D03 4.67 mm to (131.0, 26.2)
- moved D05 4.67 mm to (207.2, 26.1)
- moved D07 4.67 mm to (283.4, 26.2)
- moved D11 4.67 mm to (73.8, 26.2)
- moved D12 4.67 mm to (111.9, 26.2)
- moved D14 4.67 mm to (188.1, 26.1)
- moved D15 4.67 mm to (226.2, 26.2)
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Routing:
- net /COL3: track 220.7 -> 242.2 mm
- net /ROW1: track 468.6 -> 473.4 mm
- net Net-(D03-Pad1): track 7.99 -> 3.32 mm
- net Net-(D12-Pad1): track 7.99 -> 3.32 mm
- net Net-(D11-Pad1): track 7.99 -> 3.32 mm
- net Net-(D02-Pad1): track 7.99 -> 3.32 mm
- net Net-(D01-Pad1): track 7.99 -> 3.32 mm
- net Net-(D17-Pad1): track 7.94 -> 3.27 mm
- net Net-(D06-Pad1): track 7.94 -> 3.27 mm
- net Net-(D10-Pad1): track 7.94 -> 3.27 mm
- net Net-(D00-Pad1): track 7.94 -> 3.27 mm
- net Net-(D15-Pad1): track 7.94 -> 3.27 mm
- net Net-(D07-Pad1): track 7.94 -> 3.27 mm
- net Net-(D16-Pad1): track 7.90 -> 3.23 mm
- net Net-(D14-Pad1): track 7.89 -> 3.22 mm
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Other:
- outline, holes or cut-outs redrawn
- board text added: "0.3"
- board text removed: "0.2"
- board text removed: "USB"
- board text removed: "my usb port is too big"
