File: unix69/kicad/keybird.kicad_pcb (KiCad board)
At the start: 2 copper layers, 304.8 x 95.2 mm, 142 parts, among them SW00 ESC, SW01 2, SW02 4, SW03 6, SW04 8, SW05 0, SW06 EQUAL, SW07 BQUOT, SW10 1, SW11 3, SW12 5, SW13 7, SW14 9, SW15 MINUS, SW16 BSLSH, SW17 F13, SW20 TAB, SW21 W, SW22 R, SW23 Y, SW24 I, SW25 P, SW26 RBRAC, SW27 F14, SW30 Q, SW31 E, SW32 T, SW33 U, SW34 O, SW35 LBRAC, SW36 DEL, SW40 A, SW41 D, SW42 G, SW43 J, SW44 L, SW45 QUOTE, SW47 F15, SW50 LCTRL, SW51 S, SW52 F, SW53 H, SW54 K, SW55 COLON, SW56 RETURN, SW57 F16, SW60 LSHFT, SW61 X, SW62 V, SW63 N, SW64 COMMA, SW65 SLASH, SW66 RSHFT, SW67 UP, SW70 Z, SW71 C, SW72 B, SW73 M, SW74 DOT, SW76 LEFT, SW77 RIGHT, SW80 LFUN, SW81 LALT, SW82 LMETA, SW83 SPACE, SW84 RMETA, SW85 RCTRL, SW86 RFUN, SW87 DOWN, U1 RP2040-Tiny

Commit message: add tooling holes for pcb assembly
Parts:
- added REF**: ToolingHole_1.152mm, MountingHole:MountingHole_2.1mm, F.Cu at (317.3, 107.8)
- added REF**: ToolingHole_1.152mm, MountingHole:MountingHole_2.1mm, F.Cu at (16.1, 16.1)
Other:
- outline, holes or cut-outs redrawn
Changed lines of the file:
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@@
   )
   (setup
+    (stackup
+      (layer "F.SilkS" (type "Top Silk Screen"))
+      (layer "F.Paste" (type "Top Solder Paste"))
+      (layer "F.Mask" (type "Top Solder Mask") (color "Purple") (thickness 0.01))
+      (layer "F.Cu" (type "copper") (thickness 0.035))
+      (layer "dielectric 1" (type "core") (thickness 1.51) (material "FR4") (epsilon_r 4.5) (loss_tangent 0.02))
+      (layer "B.Cu" (type "copper") (thickness 0.035))
+      (layer "B.Mask" (type "Bottom Solder Mask") (color "Purple") (thickness 0.01))
+      (layer "B.Paste" (type "Bottom Solder Paste"))
+      (layer "B.SilkS" (type "Bottom Silk Screen"))
+      (copper_finish "None")
+      (dielectric_constraints no)
+    )
     (pad_to_mask_clearance 0)
     (pcbplotparams
@@
     )
   )
+  (footprint "MountingHole:MountingHole_2.1mm" (layer "F.Cu")
+    (at 317.301296 107.751472)
+    (descr "Mounting Hole 2.1mm, no annular")
+    (tags "mounting hole 2.1mm no annular")
+    (attr exclude_from_pos_files exclude_from_bom)
+    (fp_text reference "REF**" (at 0 -1.6) (layer "Cmts.User") hide
+      (effects (font (size 1 1) (thickness 0.15)))
+    )
+    (fp_text value "ToolingHole_1.152mm" (at 0 1.6) (layer "F.Fab")
+      (effects (font (size 1 1) (thickness 0.15)))
+    )
+    (pad "" np_thru_hole circle (at 0 0) (size 1.152 1.152) (drill 1.152) (layers F&B.Cu *.Mask)
+      (solder_mask_margin 0.074))
+    (pad "" np_thru_hole circle (at 0 0) (size 1.152 1.152) (drill 1.152) (layers F&B.Cu *.Mask)
+      (solder_mask_margin 0.074))
+  )
   (footprint "Switch_Keyboard_Hotswap_Kailh:SW_Hotswap_Kailh_MX_1.00u" (layer "F.Cu")
     (at 185.7375 42.8625)
@@
     )
   )
+  (footprint "MountingHole:MountingHole_2.1mm" (layer "F.Cu")
+    (at 16.073424 16.073424)
+    (descr "Mounting Hole 2.1mm, no annular")
+    (tags "mounting hole 2.1mm no annular")
+    (attr exclude_from_pos_files exclude_from_bom)
+    (fp_text reference "REF**" (at 0 -1.6) (layer "Cmts.User") hide
+      (effects (font (size 1 1) (thickness 0.15)))
+    )
+    (fp_text value "ToolingHole_1.152mm" (at 0 1.6) (layer "F.Fab")
+      (effects (font (size 1 1) (thickness 0.15)))
+    )
+    (pad "" np_thru_hole circle (at 0 0) (size 1.152 1.152) (drill 1.152) (layers F&B.Cu *.Mask)
+      (solder_mask_margin 0.074))
+    (pad "" np_thru_hole circle (at 0 0) (size 1.152 1.152) (drill 1.152) (layers F&B.Cu *.Mask)
+      (solder_mask_margin 0.074))
+  )
   (footprint "Diode_SMD:D_SOD-123" (layer "B.Cu")
     (at 121.443788 45.243788 90)
@@
   )
   (gr_line (start 319.0875 15.478125) (end 319.0875 108.346875) (layer "Edge.Cuts") (width 0.1))
+  (gr_arc (start 17.859628 16.668827) (mid 17.510909 17.510733) (end 16.669003 17.859452) (layer "Edge.Cuts") (width 0.1))
   (gr_arc (start 319.0875 108.346875) (mid 318.738774 109.188774) (end 317.896875 109.5375) (layer "Edge.Cuts") (width 0.1))
   (gr_arc (start 15.478125 109.5375) (mid 14.636226 109.188774) (end 14.2875 108.346875) (layer "Edge.Cuts") (width 0.1))
@@
     (effects (font (size 1.016 1.016) (thickness 0.1524)) (justify mirror))
   )
-  (gr_text "0.3" (at 164.901135 91.677893 90) (layer "B.SilkS")
+  (gr_text "0.3" (at 164.603768 91.677893 90) (layer "B.SilkS")
     (effects (font (size 1.016 1.016) (thickness 0.1524)) (justify left mirror))
   )
@@
   (segment (start 59.590056 78.422568) (end 59.5313 81.69382) (width 0.25) (layer "B.Cu") (net 80))
   (via (at 108.942279 92.868828) (size 0.8) (drill 0.4) (layers "F.Cu" "B.Cu") (net 84))
-  (via (at 16.668764 16.668764) (size 0.8) (drill 0.4) (layers "F.Cu" "B.Cu") (free) (net 84))
+  (via (at 35.71872 16.668764) (size 0.8) (drill 0.4) (layers "F.Cu" "B.Cu") (free) (net 84))
   (via (at 302.419004 16.668764) (size 0.8) (drill 0.4) (layers "F.Cu" "B.Cu") (free) (net 84))
   (via (at 35.71878 88.106324) (size 0.8) (drill 0.4) (layers "F.Cu" "B.Cu") (free) (net 84))
@@
   (via (at 302.419004 54.768796) (size 0.8) (drill 0.4) (layers "F.Cu" "B.Cu") (free) (net 84))
   (via (at 207.168924 107.15634) (size 0.8) (drill 0.4) (layers "F.Cu" "B.Cu") (free) (net 84))
-  (via (at 316.706516 107.15634) (size 0.8) (drill 0.4) (layers "F.Cu" "B.Cu") (free) (net 84))
+  (via (at 302.418496 107.15616) (size 0.8) (drill 0.4) (layers "F.Cu" "B.Cu") (free) (net 84))
   (via (at 28.71875 73.9625) (size 0.8) (drill 0.4) (layers "F.Cu" "B.Cu") (free) (net 84))
   (via (at 21.575 35.8625) (size 0.8) (drill 0.4) (layers "F.Cu" "B.Cu") (free) (net 84))

Commit message: don't need the tooling holes for jlcpcb's cheap mode
Parts:
- removed REF** (x2): ToolingHole_1.152mm, MountingHole:MountingHole_2.1mm
Changed lines of the file:
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@@
     )
     (pad_to_mask_clearance 0)
+    (grid_origin 14.2875 14.2875)
     (pcbplotparams
       (layerselection 0x00010fc_ffffffff)
@@
     )
   )
-  (footprint "MountingHole:MountingHole_2.1mm" (layer "F.Cu")
-    (at 317.301296 107.751472)
-    (descr "Mounting Hole 2.1mm, no annular")
-    (tags "mounting hole 2.1mm no annular")
-    (attr exclude_from_pos_files exclude_from_bom)
-    (fp_text reference "REF**" (at 0 -1.6) (layer "Cmts.User") hide
-      (effects (font (size 1 1) (thickness 0.15)))
-    )
-    (fp_text value "ToolingHole_1.152mm" (at 0 1.6) (layer "F.Fab")
-      (effects (font (size 1 1) (thickness 0.15)))
-    )
-    (pad "" np_thru_hole circle (at 0 0) (size 1.152 1.152) (drill 1.152) (layers F&B.Cu *.Mask)
-      (solder_mask_margin 0.074))
-    (pad "" np_thru_hole circle (at 0 0) (size 1.152 1.152) (drill 1.152) (layers F&B.Cu *.Mask)
-      (solder_mask_margin 0.074))
-  )
   (footprint "Switch_Keyboard_Hotswap_Kailh:SW_Hotswap_Kailh_MX_1.00u" (layer "F.Cu")
     (at 185.7375 42.8625)
@@
     )
   )
-  (footprint "MountingHole:MountingHole_2.1mm" (layer "F.Cu")
-    (at 16.073424 16.073424)
-    (descr "Mounting Hole 2.1mm, no annular")
-    (tags "mounting hole 2.1mm no annular")
-    (attr exclude_from_pos_files exclude_from_bom)
-    (fp_text reference "REF**" (at 0 -1.6) (layer "Cmts.User") hide
-      (effects (font (size 1 1) (thickness 0.15)))
-    )
-    (fp_text value "ToolingHole_1.152mm" (at 0 1.6) (layer "F.Fab")
-      (effects (font (size 1 1) (thickness 0.15)))
-    )
-    (pad "" np_thru_hole circle (at 0 0) (size 1.152 1.152) (drill 1.152) (layers F&B.Cu *.Mask)
-      (solder_mask_margin 0.074))
-    (pad "" np_thru_hole circle (at 0 0) (size 1.152 1.152) (drill 1.152) (layers F&B.Cu *.Mask)
-      (solder_mask_margin 0.074))
-  )
   (footprint "Diode_SMD:D_SOD-123" (layer "B.Cu")
