File: unix69/ltbs-base/ltbs-base.kicad_pcb (KiCad board)
At the start: 2 copper layers, 322.4 x 112.8 mm, 18 parts

Commit message: mounting holes for feet
Parts:
- added REF**: MountingHole_4.3mm_M4, MountingHole:MountingHole_4.3mm_M4, F.Cu at (50.1, 50.1)
- added REF**: MountingHole_4.3mm_M4, MountingHole:MountingHole_4.3mm_M4, F.Cu at (330.9, 50.1)
Other:
- outline, holes or cut-outs redrawn
Changed lines of the file:
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@@
   (paper "A3")
   (title_block
-    (title "lego technic beam sandwich - top plate")
+    (title "lego technic beam sandwich - base plate")
     (rev "0.0")
   )
@@
     (pad "" np_thru_hole circle (at 0 0) (size 5 5) (drill 5) (layers *.Cu *.Mask))
   )
+  (footprint "MountingHole:MountingHole_4.3mm_M4" (layer "F.Cu")
+    (at 330.9 50.1)
+    (descr "Mounting Hole 4.3mm, no annular, M4")
+    (tags "mounting hole 4.3mm no annular m4")
+    (attr exclude_from_pos_files exclude_from_bom)
+    (fp_text reference "REF**" (at 0 -5.3) (layer "Cmts.User") hide
+      (effects (font (size 1 1) (thickness 0.15)))
+    )
+    (fp_text value "MountingHole_4.3mm_M4" (at 0 5.3) (layer "F.Fab")
+      (effects (font (size 1 1) (thickness 0.15)))
+    )
+    (fp_circle (center 0 0) (end 4.3 0) (layer "Cmts.User") (width 0.15) (fill none))
+    (fp_circle (center 0 0) (end 4.55 0) (layer "F.CrtYd") (width 0.05) (fill none))
+    (pad "" np_thru_hole circle (at 0 0) (size 4.3 4.3) (drill 4.3) (layers *.Cu *.Mask))
+  )
   (footprint "MountingHole:MountingHole_5mm" (layer "F.Cu")
     (at 262.5 32.9)
@@
     (fp_circle (center 0 0) (end 5.25 0) (layer "F.CrtYd") (width 0.05) (fill none))
     (pad "" np_thru_hole circle (at 0 0) (size 5 5) (drill 5) (layers *.Cu *.Mask))
+  )
+  (footprint "MountingHole:MountingHole_4.3mm_M4" (layer "F.Cu")
+    (at 50.1 50.1)
+    (descr "Mounting Hole 4.3mm, no annular, M4")
+    (tags "mounting hole 4.3mm no annular m4")
+    (attr exclude_from_pos_files exclude_from_bom)
+    (fp_text reference "REF**" (at 0 -5.3) (layer "Cmts.User") hide
+      (effects (font (size 1 1) (thickness 0.15)))
+    )
+    (fp_text value "MountingHole_4.3mm_M4" (at 0 5.3) (layer "F.Fab")
+      (effects (font (size 1 1) (thickness 0.15)))
+    )
+    (fp_circle (center 0 0) (end 4.3 0) (layer "Cmts.User") (width 0.15) (fill none))
+    (fp_circle (center 0 0) (end 4.55 0) (layer "F.CrtYd") (width 0.05) (fill none))
+    (pad "" np_thru_hole circle (at 0 0) (size 4.3 4.3) (drill 4.3) (layers *.Cu *.Mask))
   )
   (footprint "MountingHole:MountingHole_5mm" (layer "F.Cu")
@@
   (gr_line (start 190.5 29) (end 190.5 24) (layer "Dwgs.User") (width 0.15))
   (gr_line (start 190.5 147.4) (end 190.5 142.4) (layer "Dwgs.User") (width 0.15))
-  (gr_line (start 341.7 29.3) (end 39.3 29.3) (layer "Edge.Cuts") (width 0.1))
+  (gr_arc (start 199.7 30.3) (mid 199.992893 29.592893) (end 200.7 29.3) (layer "Edge.Cuts") (width 0.1))
+  (gr_line (start 341.7 29.3) (end 200.7 29.3) (layer "Edge.Cuts") (width 0.1))
+  (gr_arc (start 182.3 47.5) (mid 181.592893 47.207107) (end 181.3 46.5) (layer "Edge.Cuts") (width 0.1))
+  (gr_arc (start 199.7 46.5) (mid 199.407107 47.207107) (end 198.7 47.5) (layer "Edge.Cuts") (width 0.1))
   (gr_line (start 351.7 39.3) (end 351.7 132.1) (layer "Edge.Cuts") (width 0.1))
+  (gr_line (start 199.7 30.3) (end 199.7 46.5) (layer "Edge.Cuts") (width 0.1))
   (gr_line (start 29.3 39.3) (end 29.3 132.1) (layer "Edge.Cuts") (width 0.1))
+  (gr_line (start 198.7 47.5) (end 182.3 47.5) (layer "Edge.Cuts") (width 0.1))
   (gr_arc (start 351.7 132.1) (mid 348.771068 139.171068) (end 341.7 142.1) (layer "Edge.Cuts") (width 0.1))
   (gr_line (start 39.3 142.1) (end 341.7 142.1) (layer "Edge.Cuts") (width 0.1))
   (gr_arc (start 29.3 39.3) (mid 32.228932 32.228932) (end 39.3 29.3) (layer "Edge.Cuts") (width 0.1))
   (gr_arc (start 341.7 29.3) (mid 348.771068 32.228932) (end 351.7 39.3) (layer "Edge.Cuts") (width 0.1))
+  (gr_line (start 181.3 46.5) (end 181.3 30.3) (layer "Edge.Cuts") (width 0.1))
+  (gr_arc (start 180.3 29.3) (mid 181.007107 29.592893) (end 181.3 30.3) (layer "Edge.Cuts") (width 0.1))
   (gr_arc (start 39.3 142.1) (mid 32.228932 139.171068) (end 29.3 132.1) (layer "Edge.Cuts") (width 0.1))
+  (gr_line (start 180.3 29.3) (end 39.3 29.3) (layer "Edge.Cuts") (width 0.1))
   (zone (net 0) (net_name "") (layers F&B.Cu) (hatch edge 0.508)
     (connect_pads (clearance 0.25))
