File: keybird42/pcb/keybird42.kicad_pcb (KiCad board)
At the start: 2 copper layers, 420.3 x 95.2 mm, 176 parts, among them SW111 SW_MX, SW112 SW_MX, SW113 SW_MX, SW114 SW_MX, SW115 SW_MX, SW116 SW_MX, SW117 SW_MX, SW121 SW_MX, SW122 SW_MX, SW123 SW_MX, SW124 SW_MX, SW125 SW_MX, SW126 SW_MX, SW127 SW_MX, SW131 SW_MX, SW132 SW_MX, SW133 SW_MX, SW134 SW_MX, SW135 SW_MX, SW136 SW_MX, SW137 SW_MX, SW211 SW_MX, SW212 SW_MX, SW213 SW_MX, SW214 SW_MX, SW215 SW_MX, SW216 SW_MX, SW217 SW_MX, SW221 SW_MX, SW222 SW_MX, SW223 SW_MX, SW225 SW_MX, SW226 SW_MX, SW227 SW_MX, SW231 SW_MX, SW232 SW_MX, SW233 SW_MX, SW234 SW_MX, SW235 SW_MX, SW236 SW_MX, SW237 SW_MX, SW311 SW_MX, SW312 SW_MX, SW314 SW_MX, SW315 SW_MX, SW316 SW_MX, SW317 SW_MX, SW321 SW_MX, SW322 SW_MX, SW323 SW_MX, SW324 SW_MX, SW325 SW_MX, SW327 SW_MX, SW331 SW_MX, SW332 SW_MX, SW333 SW_MX, SW334 SW_MX, SW335 SW_MX, SW336 SW_MX, SW337 SW_MX, SW411 SW_MX, SW412 SW_MX, SW413 SW_MX, SW414 SW_MX, SW415 SW_MX, SW416 SW_MX, SW417 SW_MX, SW421 SW_MX, SW423 SW_MX, SW424 SW_MX, SW425 SW_MX, SW426 SW_MX, SW427 SW_MX, SW431 SW_MX, SW432 SW_MX, SW433 SW_MX, SW434 SW_MX, SW436 SW_MX, SW437 SW_MX, SW501 SW_MX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

Commit message: fix DRC errors
Connections:
- U1 pad 1: /ROW12 -> /COL1
- U1 pad 10: /ROW42 -> /ROW41
- U1 pad 11: /ROW43 -> /ROW42
- U1 pad 12: /ROW50 -> /ROW43
- U1 pad 13: /COL1 -> /ROW50
- U1 pad 14: /COL2 -> /COL3
- U1 pad 15: /COL3 -> /COL5
- U1 pad 16: /COL4 -> /ROW31
- U1 pad 17: /COL5 -> /ROW21
- U1 pad 18: /COL6 -> /ROW23
- U1 pad 19: /COL7 -> /ROW13
- U1 pad 2: /ROW13 -> /COL7
- U1 pad 3: /ROW21 -> /ROW12
- U1 pad 5: /ROW23 -> /COL6
- U1 pad 6: /ROW31 -> /COL2
- U1 pad 9: /ROW41 -> /COL4
Routing:
- net Net-(D505-A): track 0.00 -> 3.60 mm
- net Net-(D501-A): track 0.00 -> 3.60 mm
- net Net-(D506-A): track 0.00 -> 3.60 mm
- net Net-(D504-A): track 0.00 -> 3.60 mm
Changed lines of the file:
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@@
         (effects (font (size 1 1) (thickness 0.15)))
     )
+    (fp_line (start -11.8 -9) (end -11.8 9)
+      (stroke (width 0.1) (type default)) (layer "B.SilkS"))
+    (fp_line (start -11.8 -9) (end -11 -9)
+      (stroke (width 0.1) (type default)) (layer "B.SilkS"))
+    (fp_line (start -11.8 9) (end -11 9)
+      (stroke (width 0.1) (type default)) (layer "B.SilkS"))
     (fp_line (start -8.255 5.08) (end -6.985 5.08)
       (stroke (width 0.1) (type default)) (layer "B.SilkS"))
@@
     (fp_line (start -7.62 5.715) (end -7.62 5.08)
       (stroke (width 0.1) (type default)) (layer "B.SilkS"))
-    (fp_rect (start -11.75 -9) (end 11.75 9)
-      (stroke (width 0.1) (type default)) (fill none) (layer "B.SilkS"))
+    (fp_line (start 11 9) (end 11.8 9)
+      (stroke (width 0.1) (type default)) (layer "B.SilkS"))
+    (fp_line (start 11.8 -9) (end 11 -9)
+      (stroke (width 0.1) (type default)) (layer "B.SilkS"))
+    (fp_line (start 11.8 -9) (end 11.8 -6)
+      (stroke (width 0.1) (type default)) (layer "B.SilkS"))
+    (fp_line (start 11.8 9) (end 11.8 6)
+      (stroke (width 0.1) (type default)) (layer "B.SilkS"))
     (fp_circle (center -10.16 -5.08) (end -9.525 -5.08)
       (stroke (width 0.1) (type solid)) (fill solid) (layer "B.SilkS"))
@@
       (net 1 "/ROW11") (pinfunction "GPIO0") (pintype "bidirectional"))
     (pad "1" smd roundrect (at -7.62 -8.255) (size 1.27 3.81) (layers "B.Cu" "B.Paste" "B.Mask") (roundrect_rratio 0.2)
-      (net 9 "/ROW12") (pinfunction "GPIO1") (pintype "bidirectional"))
+      (net 100 "/COL1") (pinfunction "GPIO1") (pintype "bidirectional"))
     (pad "2" smd roundrect (at -5.08 -8.255) (size 1.27 3.81) (layers "B.Cu" "B.Paste" "B.Mask") (roundrect_rratio 0.2)
-      (net 17 "/ROW13") (pinfunction "GPIO2") (pintype "bidirectional"))
+      (net 106 "/COL7") (pinfunction "GPIO2") (pintype "bidirectional"))
     (pad "3" smd roundrect (at -2.54 -8.255) (size 1.27 3.81) (layers "B.Cu" "B.Paste" "B.Mask") (roundrect_rratio 0.2)
-      (net 25 "/ROW21") (pinfunction "GPIO3") (pintype "bidirectional"))
+      (net 9 "/ROW12") (pinfunction "GPIO3") (pintype "bidirectional"))
     (pad "4" smd roundrect (at 0 -8.255) (size 1.27 3.81) (layers "B.Cu" "B.Paste" "B.Mask") (roundrect_rratio 0.2)
       (net 33 "/ROW22") (pinfunction "GPIO4") (pintype "bidirectional"))
     (pad "5" smd roundrect (at 2.54 -8.255) (size 1.27 3.81) (layers "B.Cu" "B.Paste" "B.Mask") (roundrect_rratio 0.2)
-      (net 40 "/ROW23") (pinfunction "GPIO5") (pintype "bidirectional"))
+      (net 105 "/COL6") (pinfunction "GPIO5") (pintype "bidirectional"))
     (pad "6" smd roundrect (at 5.08 -8.255) (size 1.27 3.81) (layers "B.Cu" "B.Paste" "B.Mask") (roundrect_rratio 0.2)
-      (net 48 "/ROW31") (pinfunction "GPIO6") (pintype "bidirectional"))
+      (net 101 "/COL2") (pinfunction "GPIO6") (pintype "bidirectional"))
     (pad "7" smd roundrect (at 7.62 -8.255) (size 1.27 3.81) (layers "B.Cu" "B.Paste" "B.Mask") (roundrect_rratio 0.2)
       (net 56 "/ROW32") (pinfunction "GPIO7") (pintype "bidirectional"))
@@
       (net 63 "/ROW33") (pinfunction "GPIO8") (pintype "bidirectional"))
     (pad "9" smd roundrect (at 10.795 -5.08 90) (size 1.27 3.81) (layers "B.Cu" "B.Paste" "B.Mask") (roundrect_rratio 0.2)
-      (net 71 "/ROW41") (pinfunction "GPIO9") (pintype "bidirectional"))
+      (net 103 "/COL4") (pinfunction "GPIO9") (pintype "bidirectional"))
     (pad "10" smd roundrect (at 10.795 -2.54 90) (size 1.27 3.81) (layers "B.Cu" "B.Paste" "B.Mask") (roundrect_rratio 0.2)
-      (net 79 "/ROW42") (pinfunction "GPIO10") (pintype "bidirectional"))
+      (net 71 "/ROW41") (pinfunction "GPIO10") (pintype "bidirectional"))
     (pad "11" smd roundrect (at 10.795 0 90) (size 1.27 3.81) (layers "B.Cu" "B.Paste" "B.Mask") (roundrect_rratio 0.2)
-      (net 86 "/ROW43") (pinfunction "GPIO11") (pintype "bidirectional"))
+      (net 79 "/ROW42") (pinfunction "GPIO11") (pintype "bidirectional"))
     (pad "12" smd roundrect (at 10.795 2.54 90) (size 1.27 3.81) (layers "B.Cu" "B.Paste" "B.Mask") (roundrect_rratio 0.2)
-      (net 92 "/ROW50") (pinfunction "GPIO12") (pintype "bidirectional"))
+      (net 86 "/ROW43") (pinfunction "GPIO12") (pintype "bidirectional"))
     (pad "13" smd roundrect (at 10.795 5.08 90) (size 1.27 3.81) (layers "B.Cu" "B.Paste" "B.Mask") (roundrect_rratio 0.2)
-      (net 100 "/COL1") (pinfunction "GPIO13") (pintype "bidirectional"))
+      (net 92 "/ROW50") (pinfunction "GPIO13") (pintype "bidirectional"))
     (pad "14" smd roundrect (at 10.16 8.255 180) (size 1.27 3.81) (layers "B.Cu" "B.Paste" "B.Mask") (roundrect_rratio 0.2)
-      (net 101 "/COL2") (pinfunction "GPIO14") (pintype "bidirectional"))
+      (net 102 "/COL3") (pinfunction "GPIO14") (pintype "bidirectional"))
     (pad "15" smd roundrect (at 7.62 8.255 180) (size 1.27 3.81) (layers "B.Cu" "B.Paste" "B.Mask") (roundrect_rratio 0.2)
-      (net 102 "/COL3") (pinfunction "GPIO15") (pintype "bidirectional"))
+      (net 104 "/COL5") (pinfunction "GPIO15") (pintype "bidirectional"))
     (pad "16" smd roundrect (at 5.08 8.255 180) (size 1.27 3.81) (layers "B.Cu" "B.Paste" "B.Mask") (roundrect_rratio 0.2)
-      (net 103 "/COL4") (pinfunction "GPIO26") (pintype "bidirectional"))
+      (net 48 "/ROW31") (pinfunction "GPIO26") (pintype "bidirectional"))
     (pad "17" smd roundrect (at 2.54 8.255 180) (size 1.27 3.81) (layers "B.Cu" "B.Paste" "B.Mask") (roundrect_rratio 0.2)
-      (net 104 "/COL5") (pinfunction "GPIO27") (pintype "bidirectional"))
+      (net 25 "/ROW21") (pinfunction "GPIO27") (pintype "bidirectional"))
     (pad "18" smd roundrect (at 0 8.255 180) (size 1.27 3.81) (layers "B.Cu" "B.Paste" "B.Mask") (roundrect_rratio 0.2)
-      (net 105 "/COL6") (pinfunction "GPIO28") (pintype "bidirectional"))
+      (net 40 "/ROW23") (pinfunction "GPIO28") (pintype "bidirectional"))
     (pad "19" smd roundrect (at -2.54 8.255 180) (size 1.27 3.81) (layers "B.Cu" "B.Paste" "B.Mask") (roundrect_rratio 0.2)
-      (net 106 "/COL7") (pinfunction "GPIO29") (pintype "bidirectional"))
+      (net 17 "/ROW13") (pinfunction "GPIO29") (pintype "bidirectional"))
     (pad "20" smd roundrect (at -5.08 8.255 180) (size 1.27 3.81) (layers "B.Cu" "B.Paste" "B.Mask") (roundrect_rratio 0.2)
       (net 107 "unconnected-(U1-3v3-Pad20)") (pinfunction "3v3") (pintype "power_out+no_connect"))
@@
   (arc (start 317.896875 103.585106) (mid 317.896945 103.584758) (end 317.897142 103.584462) (width 0.254) (layer "B.Cu") (net 92))
   (arc (start 344.090625 103.585159) (mid 344.0907 103.584782) (end 344.090914 103.584462) (width 0.254) (layer "B.Cu") (net 92))
+  (segment (start 103.47325 99.695) (end 103.87625 99.695) (width 0.254) (layer "B.Cu") (net 93))
+  (arc (start 103.87625 99.695) (mid 105.353661 100.306964) (end 105.965625 101.784375) (width 0.254) (layer "B.Cu") (net 93))
   (segment (start 127.28575 99.695) (end 127.68875 99.695) (width 0.254) (layer "B.Cu") (net 94))
   (arc (start 127.68875 99.695) (mid 129.166161 100.306964) (end 129.778125 101.784375) (width 0.254) (layer "B.Cu") (net 94))
   (segment (start 153.4795 99.695) (end 153.8825 99.695) (width 0.254) (layer "B.Cu") (net 95))
   (arc (start 153.8825 99.695) (mid 155.359911 100.306964) (end 155.971875 101.784375) (width 0.254) (layer "B.Cu") (net 95))
+  (segment (start 234.442 99.695) (end 234.845 99.695) (width 0.254) (layer "B.Cu") (net 96))
+  (arc (start 234.845 99.695) (mid 236.322411 100.306964) (end 236.934375 101.784375) (width 0.254) (layer "B.Cu") (net 96))
+  (segment (start 315.4045 99.695) (end 315.8075 99.695) (width 0.254) (layer "B.Cu") (net 97))
+  (arc (start 315.8075 99.695) (mid 317.284911 100.306964) (end 317.896875 101.784375) (width 0.254) (layer "B.Cu") (net 97))
+  (segment (start 341.59825 99.695) (end 342.00125 99.695) (width 0.254) (layer "B.Cu") (net 98))
+  (arc (start 342.00125 99.695) (mid 343.478661 100.306964) (end 344.090625 101.784375) (width 0.254) (layer "B.Cu") (net 98))
   (segment (start 365.41075 99.695) (end 365.81375 99.695) (width 0.254) (layer "B.Cu") (net 99))
   (arc (start 365.81375 99.695) (mid 367.291161 100.306964) (end 367.903125 101.784375) (width 0.254) (layer "B.Cu") (net 99))

Commit message: add a caption
Other:
- board text added: "Tony Finch <dot@dotat.at>"
- board text added: "designed and assembled"
- board text added: "in Cambridge by"
- board text added: "keybird 42"
Changed lines of the file:
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@@
   (gr_line (start 166.6875 114.3) (end 290.5125 114.3)
     (stroke (width 0.1) (type default)) (layer "Edge.Cuts"))
+  (gr_text "designed and assembled" (at 197.643916 105.370401) (layer "B.SilkS")
+    (effects (font (size 1.190625 1.190625) (thickness 0.148828)) (justify bottom mirror))
+  )
+  (gr_text "Tony Finch <dot@dotat.at>" (at 197.643916 111.918844) (layer "B.SilkS")
+    (effects (font (size 1.5875 1.5875) (thickness 0.198438)) (justify bottom mirror))
+  )
+  (gr_text "in Cambridge by" (at 197.643916 107.751653) (layer "B.SilkS")
+    (effects (font (size 1.190625 1.190625) (thickness 0.148828)) (justify bottom mirror))
+  )
+  (gr_text "keybird 42" (at 197.643916 101.20321) (layer "B.SilkS")
+    (effects (font (size 4.7625 4.7625) (thickness 0.595313) italic) (justify bottom mirror))
+  )
   (segment (start 217.884558 26.789085) (end 217.884558 32.146902) (width 0.254) (layer "F.Cu") (net 1))
   (segment (start 275.034606 26.789085) (end 275.034606 32.146902) (width 0.254) (layer "F.Cu") (net 1))

Commit message: fiddling with iobird track routing
Parts:
- added J1: IObird FPC, Connector_FFC-FPC:Hirose_FH12-40S-0.5SH_1x40-1MP_P0.50mm_Horizontal, B.Cu at (251.8, 104.2)
- moved U1 6.55 mm to (268.5, 103.6)
Routing:
- net /ROW12: track 561.8 -> 546.7 mm
- net /ROW13: track 556.1 -> 542.0 mm
- net /ROW11: track 563.8 -> 551.6 mm
- net /ROW33: track 505.1 -> 516.3 mm
- net /COL5: track 706.0 -> 715.6 mm
- net /COL7: track 758.2 -> 749.3 mm
- net /ROW32: track 505.4 -> 514.0 mm
- net /COL4: track 679.6 -> 671.8 mm
- net /ROW50: track 557.5 -> 549.6 mm
- net /ROW42: track 494.0 -> 486.4 mm
- net /ROW43: track 494.2 -> 487.7 mm
- net /ROW41: track 504.1 -> 497.8 mm
- net /COL3: track 708.1 -> 714.3 mm
- net /COL1: track 808.7 -> 802.7 mm
- net /ROW31: track 512.6 -> 518.2 mm
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